File: 1_PCB/1_PCB/V0.2/TimeTracker_TestboardV1.brd (EAGLE design)
At the start: 105.1 x 80 mm, 47 parts, among them IC1 L78L33ABUTR, IC2 7805DT, IC3 PCF8574T_3,518, IC4 PCF8574T_3,518, U1 WS2812B, U2 WS2812B, U3 WS2812B, U4 WS2812B, U5 SMTM1225, Y1 FX135A-327

Commit message: Nicolas
PCB Update
Parts:
- removed C1: (no value), rcl:C0805
- added 0.1µ: (no value), rcl:C0805
- added RESET: (no value), jumper:JP1
- C2, C6, C8: value (none) -> 0,1µ
- moved V_IN 1.27 mm to (8.89, 73.7)
- moved JP7 1.27 mm to (97.8, 48.3)
- moved C4 1.02 mm to (6.86, 66.0), turned to 180 degrees
- moved C2 0.38 mm to (24.4, 74.9)
- renumbered JP5 to VCC_µC
Connections:
- net GND: now also 0.1µ.2, RESET.1; no longer C1.2
- net GND1: now also RESET.2
- net N$1: now also 0.1µ.1; no longer C1.1
Routing:
- net GND1: track 11.3 -> 16.5 mm
- net GND: track 92.9 -> 97.7 mm, vias 14 -> 16
- net I2CSDA: track 131.4 -> 133.5 mm
- net RFID_CS: track 73.4 -> 75.2 mm
- net 3V3: track 401.3 -> 399.8 mm
- net SPISCK: track 155.1 -> 153.6 mm, vias 2 -> 4
- net SPIMOSI: track 157.8 -> 156.5 mm
- net DISPLAY_RESET: track 34.0 -> 32.7 mm
- net DISPLAY_DC: track 38.1 -> 36.8 mm
- net DISPLAY_CS: track 43.0 -> 41.7 mm
Other:
- board size 105.1 x 80 mm -> 102.9 x 78.8 mm
- board text added: "2x 10K"
- board text added: "3v3"
- board text added: "3x 10K"
- board text added: "4x 0.1µ"
- board text added: "4x100K"
- board text added: "CS"
- board text added: "DC"
- board text added: "GND"
- board text added: "MISO"
- board text added: "MOSI"
- board text added: "Reset"
- board text added: "SCK"

Commit message: Nicolas
Update PCB Ready for Production
Parts:
- added R14, R15: 10K, rcl:R0805
Connections:
- net 3V3: now also R14.1, R15.1
- net I2CSCL: now also R14.2
- net I2CSDA: now also R15.2
Routing:
- net I2CSDA: track 133.5 -> 151.2 mm, vias 3 -> 5
- net GND: track 97.7 -> 111.5 mm
- net I2CSCL: track 139.8 -> 152.6 mm, vias 3 -> 5
- net 3V3: track 399.8 -> 411.5 mm
- net 5V: track 97.6 -> 97.1 mm
Other:
- board size 102.9 x 78.8 mm -> 104.2 x 78.8 mm
- board text added: "2x10K"
Changed lines of the file:
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@@
 <wire x1="46.99" y1="5.08" x2="52.07" y2="5.08" width="0" layer="20"/>
 <wire x1="52.07" y1="5.08" x2="57.15" y2="0" width="0" layer="20"/>
-<wire x1="57.15" y1="0" x2="95.25" y2="0" width="0" layer="20"/>
-<wire x1="95.25" y1="0" x2="100.381" y2="7.588525" width="0" layer="20"/>
-<wire x1="100.381" y1="7.588525" x2="100.381" y2="70.983" width="0" layer="20"/>
-<wire x1="100.381" y1="70.983" x2="93.916525" y2="77.502415625" width="0" layer="20"/>
+<wire x1="57.15" y1="0" x2="92.71" y2="0" width="0" layer="20"/>
+<wire x1="92.71" y1="0" x2="101.651" y2="7.588525" width="0" layer="20"/>
+<wire x1="101.651" y1="7.588525" x2="101.651" y2="70.983" width="0" layer="20"/>
+<wire x1="101.651" y1="70.983" x2="93.916525" y2="77.502415625" width="0" layer="20"/>
 <wire x1="93.916525" y1="77.502415625" x2="-2.54" y2="77.46" width="0" layer="20"/>
 <wire x1="-2.54" y1="77.46" x2="-2.54" y2="53.34" width="0" layer="20"/>
@@
 <text x="2.54" y="12.7" size="1.27" layer="25" rot="R90">4x100K</text>
 <text x="22.86" y="52.07" size="1.778" layer="25">2x 10K</text>
+<text x="72.39" y="15.24" size="1.778" layer="25">2x10K</text>
 </plain>
 <attributes>
@@
 <attribute name="VALUE" x="25.781" y="22.86" size="1.27" layer="27" ratio="10" rot="R90"/>
 </element>
+<element name="R14" library="rcl" library_urn="urn:adsk.eagle:library:334" package="R0805" package3d_urn="urn:adsk.eagle:package:23553/2" value="10K" x="72.39" y="19.05" smashed="yes" rot="R270">
+<attribute name="POPULARITY" value="86" x="72.39" y="19.05" size="1.778" layer="27" rot="R270" display="off"/>
+<attribute name="SPICEPREFIX" value="R" x="72.39" y="19.05" size="1.778" layer="27" rot="R270" display="off"/>
+</element>
+<element name="R15" library="rcl" library_urn="urn:adsk.eagle:library:334" package="R0805" package3d_urn="urn:adsk.eagle:package:23553/2" value="10K" x="76.2" y="19.05" smashed="yes" rot="R270">
+<attribute name="POPULARITY" value="86" x="76.2" y="19.05" size="1.778" layer="27" rot="R270" display="off"/>
+<attribute name="SPICEPREFIX" value="R" x="76.2" y="19.05" size="1.778" layer="27" rot="R270" display="off"/>
+</element>
 </elements>
 <signals>
@@
 <wire x1="47.24263125" y1="6.985" x2="40.15603125" y2="-0.1016" width="0.3048" layer="1"/>
 <wire x1="24.36" y1="71.325" x2="24.36" y2="73.956" width="0.3048" layer="1"/>
-<wire x1="87.249" y1="33.462" x2="84.201" y2="33.462" width="0" layer="19" extent="1-1"/>
+<wire x1="87.249" y1="33.462" x2="84.201" y2="33.462" width="0.1524" layer="1"/>
+<contactref element="R14" pad="1"/>
+<contactref element="R15" pad="1"/>
+<wire x1="72.39" y1="20" x2="76.2" y2="20" width="0.1524" layer="1"/>
+<wire x1="72.39" y1="20" x2="69.85" y2="22.54" width="0.1524" layer="1"/>
+<wire x1="69.85" y1="22.54" x2="68.58" y2="22.54" width="0.1524" layer="1"/>
 </signal>
 <signal name="GND">
@@
 <contactref element="U3" pad="3"/>
 <contactref element="U4" pad="3"/>
-<polygon width="0.1524" layer="1" isolate="0.3048">
+<polygon width="0.1524" layer="1" isolate="0.4064">
 <vertex x="10.16" y="92.71"/>
 <vertex x="87.23923125" y="92.71"/>
@@
 <wire x1="16.256" y1="13.716" x2="16.891" y2="14.351" width="0.3048" layer="16"/>
 <wire x1="16.891" y1="14.351" x2="16.891" y2="23.876" width="0.3048" layer="16"/>
-<via x="84.455" y="24.638" extent="1-16" drill="0.35"/>
+<via x="81.915" y="32.258" extent="1-16" drill="0.35"/>
 <via x="84.455" y="21.336" extent="1-16" drill="0.35"/>
-<wire x1="84.455" y1="24.638" x2="84.455" y2="23.241" width="0.3048" layer="16"/>
 <wire x1="84.455" y1="23.241" x2="84.455" y2="21.336" width="0.3048" layer="16"/>
 <wire x1="85.6742" y1="28.575" x2="85.9409" y2="28.3083" width="0.1524" layer="1"/>
 <wire x1="85.9409" y1="28.3083" x2="85.9409" y2="27.8453125" width="0.1524" layer="1"/>
-<wire x1="85.9409" y1="27.8453125" x2="86.3542125" y2="27.432" width="0.1524" layer="1"/>
+<wire x1="85.9409" y1="27.8453125" x2="86.10310625" y2="27.68310625" width="0.1524" layer="1"/>
+<wire x1="86.10310625" y1="27.68310625" x2="86.3542125" y2="27.432" width="0.1524" layer="1"/>
 <wire x1="86.3542125" y1="27.432" x2="87.122" y2="27.432" width="0.1524" layer="1"/>
 <wire x1="87.122" y1="27.432" x2="88.138" y2="26.416" width="0.1524" layer="1"/>
@@
 <wire x1="86.614" y1="23.368" x2="86.487" y2="23.241" width="0.1524" layer="16"/>
 <wire x1="86.487" y1="23.241" x2="84.455" y2="23.241" width="0.1524" layer="16"/>
+<wire x1="84.455" y1="23.241" x2="82.169" y2="23.241" width="0.1524" layer="16"/>
+<wire x1="82.169" y1="23.241" x2="81.915" y2="23.241" width="0.1524" layer="16"/>
 <wire x1="72.8472" y1="9.525" x2="72.2122" y2="8.89" width="0.1524" layer="1"/>
 <wire x1="72.2122" y1="8.89" x2="64.77" y2="8.89" width="0.1524" layer="1"/>
@@
 <wire x1="59.436" y1="63.754" x2="60.706" y2="63.754" width="0.1524" layer="16"/>
 <wire x1="60.706" y1="63.754" x2="63.246" y2="66.294" width="0.1524" layer="16"/>
+<wire x1="81.915" y1="32.258" x2="80.01" y2="30.353" width="0.1524" layer="16"/>
+<wire x1="80.01" y1="30.353" x2="80.01" y2="25.4" width="0.1524" layer="16"/>
+<wire x1="80.01" y1="25.4" x2="82.169" y2="23.241" width="0.1524" layer="16"/>
+<wire x1="85.4202" y1="26.035" x2="85.4202" y2="27.0002" width="0.1524" layer="1"/>
+<wire x1="85.4202" y1="27.0002" x2="86.10310625" y2="27.68310625" width="0.1524" layer="1"/>
 </signal>
 <signal name="RFID_RESET">
@@
 <wire x1="7.88" y1="63.22" x2="7.874" y2="63.226" width="0.3048" layer="1"/>
 <wire x1="29.21" y1="31.75" x2="29.21" y2="29.337" width="0.3048" layer="16"/>
-<wire x1="33.401" y1="25.146" x2="33.401" y2="23.1748875" width="0.3048" layer="16"/>
-<wire x1="33.401" y1="23.1748875" x2="32.7914" y2="22.5652875" width="0.3048" layer="16"/>
-<wire x1="32.7914" y1="22.5652875" x2="32.7914" y2="21.6815125" width="0.3048" layer="16"/>
-<wire x1="32.7914" y1="21.6815125" x2="33.401" y2="21.0719125" width="0.3048" layer="16"/>
-<wire x1="33.401" y1="21.0719125" x2="33.401" y2="10.668" width="0.3048" layer="16"/>
-<wire x1="29.21" y1="29.337" x2="33.401" y2="25.146" width="0.3048" layer="16"/>
+<wire x1="31.5214" y1="27.0256" x2="31.5214" y2="21.6815125" width="0.3048" layer="16"/>
+<wire x1="31.5214" y1="21.6815125" x2="33.401" y2="19.8019125" width="0.3048" layer="16"/>
+<wire x1="33.401" y1="19.8019125" x2="33.401" y2="10.668" width="0.3048" layer="16"/>
+<wire x1="29.21" y1="29.337" x2="31.5214" y2="27.0256" width="0.3048" layer="16"/>
 <wire x1="7.88" y1="63.22" x2="7.808" y2="63.292" width="0.3048" layer="1"/>
 <wire x1="7.808" y1="63.292" x2="7.808" y2="66.04" width="0.3048" layer="1"/>
@@
 <wire x1="60.96" y1="20.32" x2="63.5" y2="22.86" width="0.1524" layer="1"/>
 <via x="63.5" y="22.86" extent="1-16" drill="0.35"/>
-<wire x1="68.935" y1="27.305" x2="67.945" y2="27.305" width="0.1524" layer="1"/>
+<wire x1="68.935" y1="27.305" x2="68.58" y2="27.305" width="0.1524" layer="1"/>
+<wire x1="68.58" y1="27.305" x2="67.945" y2="27.305" width="0.1524" layer="1"/>
 <wire x1="67.945" y1="27.305" x2="63.5" y2="22.86" width="0.1524" layer="1"/>
+<contactref element="R15" pad="2"/>
+<wire x1="76.2" y1="18.1" x2="77.79" y2="18.1" width="0.1524" layer="1"/>
+<wire x1="77.79" y1="18.1" x2="78.74" y2="19.05" width="0.1524" layer="1"/>
+<via x="78.74" y="19.05" extent="1-16" drill="0.35"/>
+<wire x1="78.74" y1="19.05" x2="78.74" y2="21.59" width="0.1524" layer="16"/>
+<via x="72.644" y="27.305" extent="1-16" drill="0.35"/>
+<wire x1="72.644" y1="27.305" x2="68.935" y2="27.305" width="0.1524" layer="1"/>
+<wire x1="78.74" y1="21.59" x2="73.025" y2="27.305" width="0.1524" layer="16"/>
+<wire x1="73.025" y1="27.305" x2="72.644" y2="27.305" width="0.1524" layer="16"/>
 </signal>
 <signal name="I2CSCL">
@@
 <wire x1="57.505" y1="9.525" x2="59.055" y2="9.525" width="0.1524" layer="1"/>
 <wire x1="59.055" y1="9.525" x2="59.69" y2="10.16" width="0.1524" layer="1"/>
-<wire x1="59.69" y1="10.16" x2="59.69" y2="25.4" width="0.1524" layer="1"/>
+<wire x1="59.69" y1="10.16" x2="59.69" y2="17.78" width="0.1524" layer="1"/>
 <via x="59.69" y="27.94" extent="1-16" drill="0.35"/>
+<wire x1="59.69" y1="17.78" x2="59.69" y2="25.4" width="0.1524" layer="1"/>
 <wire x1="59.69" y1="25.4" x2="59.69" y2="27.94" width="0.1524" layer="1"/>
 <wire x1="59.69" y1="27.94" x2="59.69" y2="31.75" width="0.1524" layer="16"/>
@@
 <wire x1="68.935" y1="28.575" x2="62.865" y2="28.575" width="0.1524" layer="1"/>
 <wire x1="60.0202" y1="60.706" x2="60.96" y2="61.6458" width="0.1524" layer="1"/>
+<contactref element="R14" pad="2"/>
+<wire x1="72.39" y1="18.1" x2="70.17" y2="18.1" width="0.1524" layer="1"/>
+<wire x1="70.17" y1="18.1" x2="69.85" y2="17.78" width="0.1524" layer="1"/>
+<via x="69.85" y="17.78" extent="1-16" drill="0.35"/>
+<wire x1="69.85" y1="17.78" x2="59.69" y2="17.78" width="0.1524" layer="16"/>
+<via x="59.69" y="17.78" extent="1-16" drill="0.35"/>
 </signal>
 <signal name="LED_DIN">
@@
 <contactref element="IC4" pad="1"/>
 <contactref element="SJ1" pad="2"/>
-<wire x1="80.645" y1="26.035" x2="81.28" y2="25.4" width="0.1524" layer="1"/>
-<wire x1="81.28" y1="25.4" x2="82.931" y2="25.4" width="0.1524" layer="1"/>
-<wire x1="82.931" y1="25.4" x2="84.709" y2="27.178" width="0.1524" layer="1"/>
-<wire x1="84.709" y1="27.178" x2="85.979" y2="27.178" width="0.1524" layer="1"/>
-<wire x1="85.979" y1="27.178" x2="86.233" y2="26.924" width="0.1524" layer="1"/>
-<wire x1="86.233" y1="26.924" x2="86.233" y2="26.035" width="0.1524" layer="1"/>
+<wire x1="81.28" y1="25.4" x2="80.645" y2="26.035" width="0.1524" layer="1"/>
 <wire x1="78.385" y1="26.035" x2="80.645" y2="26.035" width="0.1524" layer="1"/>
+<wire x1="86.233" y1="26.035" x2="86.233" y2="25.273" width="0.1524" layer="1"/>
+<wire x1="86.233" y1="25.273" x2="85.725" y2="24.765" width="0.1524" layer="1"/>
+<wire x1="84.328" y1="24.765" x2="83.693" y2="25.4" width="0.1524" layer="1"/>
+<wire x1="85.725" y1="24.765" x2="84.328" y2="24.765" width="0.1524" layer="1"/>
+<wire x1="83.693" y1="25.4" x2="81.28" y2="25.4" width="0.1524" layer="1"/>
 </signal>
 <signal name="N$18">
