File: 1_PCB/1_PCB/V0.2/TimeTracker_TestboardV1.sch (EAGLE design)
At the start: 47 parts, among them IC1 L78L33ABUTR, IC2 7805DT, IC3 PCF8574T_3,518, IC4 PCF8574T_3,518, U1 WS2812B, U2 WS2812B, U3 WS2812B, U4 WS2812B, U5 SMTM1225, Y1 FX135A-327

Commit message: Nicolas
PCB Update
Parts:
- added RESET: (no value), jumper:JP1Q
- C2, C6, C8: value (none) -> 0,1µ
- renumbered C1 to 0.1µ, JP5 to VCC_µC
Connections:
- net GND: now also RESET.1
- net GND1: now also RESET.2
Changed lines of the file:
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@@
 <part name="U$2" library="SOP65P490X110-8N" deviceset="RTC" device=""/>
 <part name="JP1" library="pinhead" library_urn="urn:adsk.eagle:library:325" deviceset="PINHD-1X8" device="" package3d_urn="urn:adsk.eagle:package:22409/2"/>
-<part name="C1" library="rcl" library_urn="urn:adsk.eagle:library:334" deviceset="C-EU" device="C0805" package3d_urn="urn:adsk.eagle:package:23617/2"/>
-<part name="C2" library="rcl" library_urn="urn:adsk.eagle:library:334" deviceset="C-EU" device="C0805" package3d_urn="urn:adsk.eagle:package:23617/2"/>
+<part name="0.1µ" library="rcl" library_urn="urn:adsk.eagle:library:334" deviceset="C-EU" device="C0805" package3d_urn="urn:adsk.eagle:package:23617/2"/>
+<part name="C2" library="rcl" library_urn="urn:adsk.eagle:library:334" deviceset="C-EU" device="C0805" package3d_urn="urn:adsk.eagle:package:23617/2" value="0,1µ"/>
 <part name="GND1" library="supply1" library_urn="urn:adsk.eagle:library:371" deviceset="GND" device=""/>
 <part name="GND3" library="supply1" library_urn="urn:adsk.eagle:library:371" deviceset="GND" device=""/>
@@
 <part name="LED_12V1" library="led" library_urn="urn:adsk.eagle:library:259" deviceset="LED" device="SML0805" package3d_urn="urn:adsk.eagle:package:15830/1"/>
 <part name="GND36" library="supply1" library_urn="urn:adsk.eagle:library:371" deviceset="GND" device=""/>
-<part name="JP5" library="jumper" library_urn="urn:adsk.eagle:library:252" deviceset="JP1Q" device="" package3d_urn="urn:adsk.eagle:package:15455/1"/>
+<part name="VCC_µC" library="jumper" library_urn="urn:adsk.eagle:library:252" deviceset="JP1Q" device="" package3d_urn="urn:adsk.eagle:package:15455/1"/>
 <part name="Y1" library="SamacSys_Parts" deviceset="FX135A-327" device=""/>
 <part name="U5" library="SamacSys_Parts" deviceset="SMTM1225" device=""/>
@@
 <part name="R5" library="rcl" library_urn="urn:adsk.eagle:library:334" deviceset="R-EU_" device="R0805" package3d_urn="urn:adsk.eagle:package:23553/2" value="10K"/>
 <part name="R11" library="rcl" library_urn="urn:adsk.eagle:library:334" deviceset="R-EU_" device="R0805" package3d_urn="urn:adsk.eagle:package:23553/2" value="10K"/>
-<part name="C8" library="rcl" library_urn="urn:adsk.eagle:library:334" deviceset="C-EU" device="C0805" package3d_urn="urn:adsk.eagle:package:23617/2"/>
+<part name="C8" library="rcl" library_urn="urn:adsk.eagle:library:334" deviceset="C-EU" device="C0805" package3d_urn="urn:adsk.eagle:package:23617/2" value="0,1µ"/>
 <part name="GND20" library="supply1" library_urn="urn:adsk.eagle:library:371" deviceset="GND" device=""/>
 <part name="IC1" library="SamacSys_Parts" deviceset="L78L33ABUTR" device=""/>
@@
 <part name="R12" library="rcl" library_urn="urn:adsk.eagle:library:334" deviceset="R-EU_" device="R0805" package3d_urn="urn:adsk.eagle:package:23553/2" value="10K"/>
 <part name="R13" library="rcl" library_urn="urn:adsk.eagle:library:334" deviceset="R-EU_" device="R0805" package3d_urn="urn:adsk.eagle:package:23553/2" value="10K"/>
-<part name="C6" library="rcl" library_urn="urn:adsk.eagle:library:334" deviceset="C-EU" device="C0805" package3d_urn="urn:adsk.eagle:package:23617/2"/>
+<part name="C6" library="rcl" library_urn="urn:adsk.eagle:library:334" deviceset="C-EU" device="C0805" package3d_urn="urn:adsk.eagle:package:23617/2" value="0,1µ"/>
 <part name="C7" library="rcl" library_urn="urn:adsk.eagle:library:334" deviceset="C-EU" device="C0805" package3d_urn="urn:adsk.eagle:package:23617/2"/>
 <part name="JP7" library="pinhead" library_urn="urn:adsk.eagle:library:325" deviceset="PINHD-1X7" device="" package3d_urn="urn:adsk.eagle:package:22477/2"/>
 <part name="GND4" library="supply1" library_urn="urn:adsk.eagle:library:371" deviceset="GND" device=""/>
+<part name="RESET" library="jumper" library_urn="urn:adsk.eagle:library:252" deviceset="JP1Q" device="" package3d_urn="urn:adsk.eagle:package:15455/1"/>
 </parts>
 <sheets>
@@
 <attribute name="VALUE" x="-78.74" y="196.85" size="1.778" layer="96" rot="R270"/>
 </instance>
-<instance part="C1" gate="G$1" x="-190.5" y="180.34" smashed="yes">
+<instance part="0.1µ" gate="G$1" x="-190.5" y="180.34" smashed="yes">
 <attribute name="NAME" x="-188.976" y="180.721" size="1.778" layer="95"/>
 <attribute name="VALUE" x="-188.976" y="175.641" size="1.778" layer="96"/>
@@
 <attribute name="VALUE" x="-203.2" y="142.24" size="1.778" layer="96"/>
 </instance>
-<instance part="JP5" gate="A" x="-25.4" y="30.48" smashed="yes">
+<instance part="VCC_µC" gate="A" x="-25.4" y="30.48" smashed="yes">
 <attribute name="NAME" x="-27.94" y="25.4" size="1.778" layer="95" rot="R90"/>
 <attribute name="VALUE" x="-20.955" y="25.4" size="1.778" layer="96" rot="R90"/>
@@
 <instance part="GND4" gate="1" x="144.78" y="119.38" smashed="yes">
 <attribute name="VALUE" x="142.24" y="116.84" size="1.778" layer="96"/>
+</instance>
+<instance part="RESET" gate="A" x="-71.12" y="43.18" smashed="yes">
+<attribute name="NAME" x="-73.66" y="38.1" size="1.778" layer="95" rot="R90"/>
+<attribute name="VALUE" x="-66.675" y="38.1" size="1.778" layer="96" rot="R90"/>
 </instance>
 </instances>
@@
 <wire x1="-149.86" y1="175.26" x2="-149.86" y2="172.72" width="0.1524" layer="91"/>
 <wire x1="-149.86" y1="172.72" x2="-172.72" y2="172.72" width="0.1524" layer="91"/>
-<pinref part="C1" gate="G$1" pin="2"/>
+<pinref part="0.1µ" gate="G$1" pin="2"/>
 <wire x1="-172.72" y1="172.72" x2="-190.5" y2="172.72" width="0.1524" layer="91"/>
 <wire x1="-190.5" y1="172.72" x2="-190.5" y2="175.26" width="0.1524" layer="91"/>
@@
 <wire x1="-58.42" y1="43.18" x2="-35.56" y2="43.18" width="0.1524" layer="91"/>
 <junction x="-35.56" y="43.18"/>
+<pinref part="RESET" gate="A" pin="1"/>
+<wire x1="-71.12" y1="35.56" x2="-71.12" y2="33.02" width="0.1524" layer="91"/>
+<wire x1="-71.12" y1="33.02" x2="-60.96" y2="33.02" width="0.1524" layer="91"/>
+<wire x1="-60.96" y1="33.02" x2="-60.96" y2="43.18" width="0.1524" layer="91"/>
+<wire x1="-60.96" y1="43.18" x2="-58.42" y2="43.18" width="0.1524" layer="91"/>
+<junction x="-58.42" y="43.18"/>
 </segment>
 <segment>
@@
 <wire x1="-208.28" y1="185.42" x2="-205.74" y2="185.42" width="0.1524" layer="91"/>
 <wire x1="-205.74" y1="185.42" x2="-205.74" y2="187.96" width="0.1524" layer="91"/>
-<pinref part="C1" gate="G$1" pin="1"/>
+<pinref part="0.1µ" gate="G$1" pin="1"/>
 <wire x1="-190.5" y1="182.88" x2="-190.5" y2="187.96" width="0.1524" layer="91"/>
 <wire x1="-190.5" y1="187.96" x2="-195.58" y2="187.96" width="0.1524" layer="91"/>
@@
 </segment>
 <segment>
-<pinref part="JP5" gate="A" pin="1"/>
+<pinref part="VCC_µC" gate="A" pin="1"/>
 <wire x1="-25.4" y1="22.86" x2="-25.4" y2="20.32" width="0.1524" layer="91"/>
 <label x="-25.4" y="20.32" size="1.778" layer="95" rot="R180" xref="yes"/>
@@
 <pinref part="U$1" gate="G$1" pin="RST"/>
 <wire x1="-38.1" y1="45.72" x2="-33.02" y2="45.72" width="0.1524" layer="91"/>
-<wire x1="-33.02" y1="45.72" x2="-20.32" y2="45.72" width="0.1524" layer="91"/>
+<wire x1="-33.02" y1="45.72" x2="-27.94" y2="45.72" width="0.1524" layer="91"/>
+<wire x1="-27.94" y1="45.72" x2="-20.32" y2="45.72" width="0.1524" layer="91"/>
 <wire x1="-33.02" y1="48.26" x2="-33.02" y2="45.72" width="0.1524" layer="91"/>
 <junction x="-33.02" y="45.72"/>
+<pinref part="RESET" gate="A" pin="2"/>
+<wire x1="-71.12" y1="50.8" x2="-71.12" y2="53.34" width="0.1524" layer="91"/>
+<wire x1="-71.12" y1="53.34" x2="-27.94" y2="53.34" width="0.1524" layer="91"/>
+<wire x1="-27.94" y1="53.34" x2="-27.94" y2="45.72" width="0.1524" layer="91"/>
+<junction x="-27.94" y="45.72"/>
 </segment>
 </net>
@@
 <net name="N$12" class="0">
 <segment>
-<pinref part="JP5" gate="A" pin="2"/>
+<pinref part="VCC_µC" gate="A" pin="2"/>
 <wire x1="-25.4" y1="38.1" x2="-25.4" y2="40.64" width="0.1524" layer="91"/>
 <pinref part="U$1" gate="G$1" pin="VIN"/>

Commit message: Nicolas
Update PCB Ready for Production
Parts:
- added R14, R15: 10K, rcl:R-EU_R0805
Connections:
- net 3V3: now also R14.1, R15.1
- net I2CSCL: now also R14.2
- net I2CSDA: now also R15.2
Changed lines of the file:
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@@
 <part name="GND4" library="supply1" library_urn="urn:adsk.eagle:library:371" deviceset="GND" device=""/>
 <part name="RESET" library="jumper" library_urn="urn:adsk.eagle:library:252" deviceset="JP1Q" device="" package3d_urn="urn:adsk.eagle:package:15455/1"/>
+<part name="R14" library="rcl" library_urn="urn:adsk.eagle:library:334" deviceset="R-EU_" device="R0805" package3d_urn="urn:adsk.eagle:package:23553/2" value="10K"/>
+<part name="R15" library="rcl" library_urn="urn:adsk.eagle:library:334" deviceset="R-EU_" device="R0805" package3d_urn="urn:adsk.eagle:package:23553/2" value="10K"/>
 </parts>
 <sheets>
@@
 <attribute name="VALUE" x="-66.675" y="38.1" size="1.778" layer="96" rot="R90"/>
 </instance>
+<instance part="R14" gate="G$1" x="246.38" y="58.42" smashed="yes" rot="R180">
+<attribute name="NAME" x="250.19" y="56.9214" size="1.778" layer="95" rot="R180"/>
+<attribute name="VALUE" x="250.19" y="61.722" size="1.778" layer="96" rot="R180"/>
+</instance>
+<instance part="R15" gate="G$1" x="246.38" y="50.8" smashed="yes" rot="R180">
+<attribute name="NAME" x="250.19" y="49.3014" size="1.778" layer="95" rot="R180"/>
+<attribute name="VALUE" x="250.19" y="54.102" size="1.778" layer="96" rot="R180"/>
+</instance>
 </instances>
 <busses>
@@
 <segment>
 <wire x1="68.58" y1="88.9" x2="78.74" y2="88.9" width="0.1524" layer="91"/>
-<label x="248.92" y="88.9" size="1.778" layer="95" xref="yes"/>
+<label x="256.54" y="88.9" size="1.778" layer="95" xref="yes"/>
 <pinref part="R4" gate="G$1" pin="2"/>
 <wire x1="78.74" y1="88.9" x2="88.9" y2="88.9" width="0.1524" layer="91"/>
@@
 <wire x1="111.76" y1="88.9" x2="121.92" y2="88.9" width="0.1524" layer="91"/>
 <wire x1="121.92" y1="88.9" x2="223.52" y2="88.9" width="0.1524" layer="91"/>
-<wire x1="223.52" y1="88.9" x2="248.92" y2="88.9" width="0.1524" layer="91"/>
+<wire x1="223.52" y1="88.9" x2="254" y2="88.9" width="0.1524" layer="91"/>
+<wire x1="254" y1="88.9" x2="256.54" y2="88.9" width="0.1524" layer="91"/>
 <wire x1="101.6" y1="83.82" x2="101.6" y2="88.9" width="0.1524" layer="91"/>
 <junction x="101.6" y="88.9"/>
@@
 <wire x1="220.98" y1="22.86" x2="220.98" y2="33.02" width="0.1524" layer="91"/>
 <junction x="220.98" y="33.02"/>
+<pinref part="R14" gate="G$1" pin="1"/>
+<wire x1="251.46" y1="58.42" x2="254" y2="58.42" width="0.1524" layer="91"/>
+<wire x1="254" y1="58.42" x2="254" y2="88.9" width="0.1524" layer="91"/>
+<junction x="254" y="88.9"/>
+<pinref part="R15" gate="G$1" pin="1"/>
+<wire x1="251.46" y1="50.8" x2="254" y2="50.8" width="0.1524" layer="91"/>
+<wire x1="254" y1="50.8" x2="254" y2="58.42" width="0.1524" layer="91"/>
+<junction x="254" y="58.42"/>
 </segment>
 <segment>
@@
 <pinref part="IC3" gate="G$1" pin="SDA"/>
 <wire x1="200.66" y1="30.48" x2="233.68" y2="30.48" width="0.1524" layer="91"/>
-<wire x1="233.68" y1="30.48" x2="233.68" y2="71.12" width="0.1524" layer="91"/>
+<wire x1="233.68" y1="30.48" x2="233.68" y2="50.8" width="0.1524" layer="91"/>
 <pinref part="IC4" gate="G$1" pin="SDA"/>
+<wire x1="233.68" y1="50.8" x2="233.68" y2="71.12" width="0.1524" layer="91"/>
 <wire x1="233.68" y1="71.12" x2="233.68" y2="81.28" width="0.1524" layer="91"/>
 <wire x1="200.66" y1="71.12" x2="233.68" y2="71.12" width="0.1524" layer="91"/>
 <junction x="233.68" y="71.12"/>
 <label x="233.68" y="81.28" size="1.778" layer="95" xref="yes"/>
+<pinref part="R15" gate="G$1" pin="2"/>
+<wire x1="241.3" y1="50.8" x2="233.68" y2="50.8" width="0.1524" layer="91"/>
+<junction x="233.68" y="50.8"/>
 </segment>
 </net>
@@
 <wire x1="236.22" y1="76.2" x2="236.22" y2="68.58" width="0.1524" layer="91"/>
 <pinref part="IC3" gate="G$1" pin="SCL"/>
-<wire x1="236.22" y1="68.58" x2="236.22" y2="27.94" width="0.1524" layer="91"/>
+<wire x1="236.22" y1="68.58" x2="236.22" y2="58.42" width="0.1524" layer="91"/>
+<wire x1="236.22" y1="58.42" x2="236.22" y2="27.94" width="0.1524" layer="91"/>
 <wire x1="236.22" y1="27.94" x2="200.66" y2="27.94" width="0.1524" layer="91"/>
 <pinref part="IC4" gate="G$1" pin="SCL"/>
@@
 <junction x="236.22" y="68.58"/>
 <label x="236.22" y="76.2" size="1.778" layer="95" xref="yes"/>
-</segment>
-</net>
+<pinref part="R14" gate="G$1" pin="2"/>
+<wire x1="241.3" y1="58.42" x2="236.22" y2="58.42" width="0.1524" layer="91"/>
+<junction x="236.22" y="58.42"/>
+</segment>
+</net>
