File: 1_PCB/1_PCB/V0.3/TimeTracker_TestboardV1.brd (EAGLE design)
At the start: 104.2 x 78.8 mm, 52 parts, among them IC1 L78L33ABUTR, IC2 7805DT, IC3 PCF8574T_3,518, IC4 PCF8574T_3,518, U1 WS2812B, U2 WS2812B, U3 WS2812B, U4 WS2812B, U5 SMTM1225, Y1 FX135A-327

Commit message: Nicolas
Update
Routing:
- net N$1: track 40.3 -> 41.5 mm
Changed lines of the file:
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@@
 <contactref element="V_IN" pad="1"/>
 <contactref element="0.1µ" pad="1"/>
-<wire x1="11.99" y1="73.66" x2="17.425" y2="68.225" width="0.6096" layer="1"/>
+<wire x1="11.99" y1="73.66" x2="12.345" y2="73.305" width="0.6096" layer="1"/>
+<wire x1="12.345" y1="73.305" x2="17.425" y2="68.225" width="0.6096" layer="1"/>
 <wire x1="12.44" y1="63.22" x2="18.06" y2="68.84" width="0.6096" layer="1"/>
 <wire x1="18.06" y1="68.84" x2="18.06" y2="68.86" width="0.6096" layer="1"/>
@@
 <wire x1="12.446" y1="63.226" x2="12.446" y2="65.217" width="0.6096" layer="1"/>
 <contactref element="R3" pad="2"/>
-<wire x1="1.27" y1="66.99" x2="7.94" y2="73.66" width="0.1524" layer="1"/>
-<wire x1="7.94" y1="73.66" x2="11.99" y2="73.66" width="0.1524" layer="1"/>
 <contactref element="IC1" pad="3"/>
 <wire x1="20.525" y1="71.325" x2="21.36" y2="71.325" width="0.508" layer="1"/>
@@
 <wire x1="21.36" y1="71.325" x2="21.36" y2="74.713" width="0.3048" layer="1"/>
 <wire x1="21.36" y1="74.713" x2="21.27" y2="74.803" width="0.3048" layer="1"/>
+<wire x1="1.27" y1="66.99" x2="1.27" y2="68.58" width="0.1524" layer="1"/>
+<wire x1="1.27" y1="68.58" x2="2.54" y2="69.85" width="0.1524" layer="1"/>
+<wire x1="2.54" y1="69.85" x2="5.08" y2="69.85" width="0.1524" layer="1"/>
+<wire x1="5.08" y1="69.85" x2="6.35" y2="71.12" width="0.1524" layer="1"/>
+<wire x1="6.35" y1="71.12" x2="8.89" y2="71.12" width="0.1524" layer="1"/>
+<wire x1="11.075" y1="73.305" x2="12.345" y2="73.305" width="0.1524" layer="1"/>
+<wire x1="8.89" y1="71.12" x2="11.075" y2="73.305" width="0.1524" layer="1"/>
 </signal>
 <signal name="5V">
